File: payload2.brd (EAGLE design)
At the start: 50.8 x 27.9 mm, 26 parts, among them U1 ATMEGA328P_TQFP, U2 USD-SOCKETSMD, U3 3.3V/150mA, U4 9DoF IMU, Y1 16MHz

Commit message: Review of payload PCB complete
Parts:
- moved Y1 1.93 mm to (19.7, 2.54), turned to 315 degrees
Routing:
- net GND: track 33.0 -> 46.3 mm, vias 7 -> 11
- net XTAL2: track 4.63 -> 2.73 mm
- net XTAL1: track 3.88 -> 2.84 mm
- net N$4: track 5.59 -> 6.52 mm
- net 3.3V: track 138.7 -> 138.1 mm
Changed lines of the file:
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@@
 <?xml version="1.0" encoding="utf-8"?>
 <!DOCTYPE eagle SYSTEM "eagle.dtd">
-<eagle version="8.3.2">
+<eagle version="9.0.0">
 <drawing>
 <settings>
@@
 <layer number="25" name="tNames" color="7" fill="1" visible="yes" active="yes"/>
 <layer number="26" name="bNames" color="7" fill="1" visible="yes" active="yes"/>
-<layer number="27" name="tValues" color="7" fill="1" visible="yes" active="yes"/>
-<layer number="28" name="bValues" color="7" fill="1" visible="yes" active="yes"/>
+<layer number="27" name="tValues" color="7" fill="1" visible="no" active="yes"/>
+<layer number="28" name="bValues" color="7" fill="1" visible="no" active="yes"/>
 <layer number="29" name="tStop" color="7" fill="3" visible="no" active="yes"/>
 <layer number="30" name="bStop" color="7" fill="6" visible="no" active="yes"/>
@@
 <layer number="43" name="vRestrict" color="2" fill="10" visible="no" active="yes"/>
 <layer number="44" name="Drills" color="7" fill="1" visible="no" active="yes"/>
-<layer number="45" name="Holes" color="7" fill="1" visible="no" active="yes"/>
+<layer number="45" name="Holes" color="7" fill="1" visible="yes" active="yes"/>
 <layer number="46" name="Milling" color="3" fill="1" visible="no" active="yes"/>
 <layer number="47" name="Measures" color="7" fill="1" visible="no" active="yes"/>
@@
 <board>
 <plain>
-<hole x="54.61" y="16.51" drill="2.1844"/>
 <hole x="3.1496" y="3.3782" drill="2.8448"/>
 <hole x="2.8702" y="25.1206" drill="2.8448"/>
@@
 <param name="dpMaxLengthDifference" value="10mm"/>
 <param name="dpGapFactor" value="2.5"/>
-<param name="checkGrid" value="0"/>
 <param name="checkAngle" value="0"/>
 <param name="checkFont" value="1"/>
 <param name="checkRestrict" value="1"/>
+<param name="checkStop" value="0"/>
+<param name="checkValues" value="0"/>
 <param name="useDiameter" value="13"/>
 <param name="maxErrors" value="50"/>
@@
 <attribute name="DIGIKEY" value="1428-1019-1-ND " x="21.59" y="20.32" size="1.778" layer="27" rot="R180" display="off"/>
 </element>
-<element name="Y1" library="femtosat" package="RESONATOR-SMD-3.2X1.3" value="16MHz" x="17.907" y="3.302" rot="R270">
-<attribute name="DIGIKEY" value="490-1198-1-ND " x="17.907" y="3.302" size="1.778" layer="27" rot="R270" display="off"/>
+<element name="Y1" library="femtosat" package="RESONATOR-SMD-3.2X1.3" value="16MHz" x="19.685" y="2.54" rot="R315">
+<attribute name="DIGIKEY" value="490-1198-1-ND " x="19.685" y="2.54" size="1.778" layer="27" rot="R315" display="off"/>
 </element>
 <element name="J7" library="SparkFun-Connectors" package="1X02" value="" x="8.2296" y="14.9098" rot="R270"/>
@@
 <wire x1="31.75" y1="8.89" x2="31.75" y2="11.938" width="0.254" layer="16"/>
 <via x="31.75" y="11.938" extent="1-16" drill="0.35"/>
-<wire x1="17.907" y1="3.302" x2="16.51" y2="3.302" width="0.254" layer="1"/>
-<wire x1="16.51" y1="3.302" x2="16.51" y2="3.81" width="0.254" layer="1"/>
 <via x="29.21" y="13.97" extent="1-16" drill="0.35"/>
 <wire x1="29.21" y1="13.97" x2="26.67" y2="13.97" width="0.381" layer="16"/>
@@
 <wire x1="5.1816" y1="18.6182" x2="1.2192" y2="18.6182" width="0.508" layer="16"/>
 <via x="1.2192" y="18.6182" extent="1-16" drill="0.4"/>
+<wire x1="19.685" y1="2.54" x2="18.415" y2="1.27" width="0.254" layer="1"/>
+<wire x1="18.415" y1="1.27" x2="17.78" y2="1.27" width="0.254" layer="1"/>
+<via x="16.51" y="1.27" extent="1-16" drill="0.508"/>
+<via x="22.86" y="1.27" extent="1-16" drill="0.508"/>
+<wire x1="16.51" y1="1.27" x2="22.86" y2="1.27" width="0.635" layer="16"/>
+<via x="15.24" y="8.89" extent="1-16" drill="0.508"/>
+<via x="21.59" y="8.89" extent="1-16" drill="0.508"/>
+<wire x1="15.24" y1="8.89" x2="21.59" y2="8.89" width="0.635" layer="16"/>
 </signal>
 <signal name="3.3V">
@@
 <wire x1="4.66" y1="16.09" x2="5.207" y2="16.0528" width="0.254" layer="1"/>
 <wire x1="23.1425" y1="19.32" x2="23.9522" y2="19.32" width="0.254" layer="1"/>
-<wire x1="23.9522" y1="21.6662" x2="23.9522" y2="21.59" width="0.254" layer="1"/>
-<wire x1="23.9522" y1="21.59" x2="23.9522" y2="19.32" width="0.254" layer="1"/>
-<wire x1="22.19" y1="21.82" x2="22.19" y2="22.5044" width="0.254" layer="1"/>
-<wire x1="22.19" y1="22.5044" x2="22.8346" y2="22.5044" width="0.254" layer="1"/>
-<wire x1="22.8346" y1="22.5044" x2="23.6728" y2="21.6662" width="0.254" layer="1"/>
-<wire x1="23.6728" y1="21.6662" x2="23.9522" y2="21.6662" width="0.254" layer="1"/>
+<wire x1="23.9522" y1="19.32" x2="23.9522" y2="21.6662" width="0.254" layer="1"/>
 <wire x1="20.0375" y1="21.32" x2="18.77375" y2="22.58375" width="0.254" layer="1"/>
 <wire x1="18.77375" y1="22.58375" x2="18.2" y2="23.1575" width="0.254" layer="1"/>
 <wire x1="18.2" y1="23.1575" x2="18.2" y2="24.13" width="0.254" layer="1"/>
-<wire x1="23.9522" y1="21.59" x2="24.2062" y2="21.844" width="0.254" layer="1"/>
-<wire x1="24.2062" y1="21.844" x2="24.2062" y2="22.3266" width="0.254" layer="1"/>
-<via x="24.2062" y="22.3266" extent="1-16" drill="0.35"/>
 <wire x1="20.5923875" y1="23.5176" x2="20.0476125" y2="23.5176" width="0.254" layer="16"/>
-<wire x1="24.2062" y1="22.3266" x2="24.0002" y2="22.5326" width="0.254" layer="16"/>
 <wire x1="19.1137625" y1="22.58375" x2="18.77375" y2="22.58375" width="0.254" layer="16"/>
 <wire x1="20.0476125" y1="23.5176" x2="19.1137625" y2="22.58375" width="0.254" layer="16"/>
@@
 <wire x1="13.4159" y1="14.9454" x2="14.898" y2="14.9454" width="0.508" layer="1"/>
 <wire x1="14.898" y1="14.9454" x2="14.898" y2="15.0114" width="0.508" layer="1"/>
+<wire x1="22.19" y1="21.82" x2="22.19" y2="22.2916" width="0.254" layer="1"/>
+<wire x1="22.19" y1="22.2916" x2="22.4282" y2="22.5298" width="0.254" layer="1"/>
+<wire x1="22.4282" y1="22.5298" x2="22.4536" y2="22.5044" width="0.254" layer="1"/>
+<wire x1="22.4536" y1="22.5044" x2="24.0002" y2="22.5044" width="0.254" layer="1"/>
+<via x="24.0002" y="22.5044" extent="1-16" drill="0.381"/>
+<wire x1="24.0002" y1="22.5044" x2="24.0002" y2="22.5326" width="0.254" layer="16"/>
+<wire x1="23.9522" y1="21.6662" x2="24.0002" y2="21.7142" width="0.254" layer="1"/>
+<wire x1="24.0002" y1="21.7142" x2="24.0002" y2="22.5044" width="0.254" layer="1"/>
 </signal>
 <signal name="MISO">
@@
 <wire x1="8.2296" y1="14.9098" x2="8.575" y2="14.92" width="0.508" layer="1"/>
 <wire x1="8.575" y1="14.92" x2="10.8157" y2="14.9454" width="0.508" layer="1"/>
-<wire x1="11.53143125" y1="14.5498" x2="11.6951" y2="14.38613125" width="0.254" layer="1"/>
-<wire x1="11.6951" y1="14.38613125" x2="11.6951" y2="13.60466875" width="0.254" layer="1"/>
-<wire x1="11.6951" y1="13.60466875" x2="11.53143125" y2="13.441" width="0.254" layer="1"/>
-<wire x1="10.8157" y1="14.9454" x2="11.2113" y2="14.5498" width="0.254" layer="1"/>
-<wire x1="11.2113" y1="14.5498" x2="11.53143125" y2="14.5498" width="0.254" layer="1"/>
-<wire x1="11.53143125" y1="13.441" x2="11.2113" y2="13.441" width="0.254" layer="1"/>
-<wire x1="11.2113" y1="13.441" x2="10.8157" y2="13.0454" width="0.254" layer="1"/>
+<wire x1="10.8157" y1="13.0454" x2="11.6738" y2="13.0454" width="0.254" layer="1"/>
+<wire x1="11.6738" y1="13.0454" x2="12.0396" y2="13.4112" width="0.254" layer="1"/>
+<wire x1="12.0396" y1="13.4112" x2="12.0396" y2="14.605" width="0.254" layer="1"/>
+<wire x1="11.6992" y1="14.9454" x2="10.8157" y2="14.9454" width="0.254" layer="1"/>
+<wire x1="12.0396" y1="14.605" x2="11.6992" y2="14.9454" width="0.254" layer="1"/>
 </signal>
 <signal name="INT">
@@
 <contactref element="Y1" pad="1"/>
 <contactref element="U1" pad="7"/>
-<wire x1="17.907" y1="4.502" x2="19.12" y2="4.502" width="0.254" layer="1"/>
-<wire x1="19.12" y1="4.502" x2="19.812" y2="3.81" width="0.254" layer="1"/>
-<wire x1="19.812" y1="3.81" x2="20.608425" y2="3.81" width="0.254" layer="1"/>
+<wire x1="18.83646875" y1="3.388528125" x2="19.257940625" y2="3.81" width="0.254" layer="1"/>
 <wire x1="20.608425" y1="3.81" x2="21.238884375" y2="4.440459375" width="0.254" layer="1"/>
+<wire x1="19.257940625" y1="3.81" x2="20.608425" y2="3.81" width="0.254" layer="1"/>
 </signal>
 <signal name="XTAL2">
 <contactref element="Y1" pad="3"/>
 <contactref element="U1" pad="8"/>
-<wire x1="17.907" y1="2.102" x2="20.0318" y2="2.102" width="0.254" layer="1"/>
-<wire x1="20.0318" y1="2.102" x2="21.804571875" y2="3.874771875" width="0.254" layer="1"/>
+<wire x1="21.781771875" y1="3.874771875" x2="21.804571875" y2="3.874771875" width="0.254" layer="1"/>
+<wire x1="21.209" y1="3.2792" x2="21.804571875" y2="3.874771875" width="0.254" layer="1"/>
+<wire x1="20.533528125" y1="1.69146875" x2="21.209" y2="2.366940625" width="0.254" layer="1"/>
+<wire x1="21.209" y1="2.366940625" x2="21.209" y2="3.2792" width="0.254" layer="1"/>
 </signal>
 <signal name="A0">
