File: payload2.brd (EAGLE design)
At the start: 50.8 x 27.9 mm, 26 parts, among them U1 ATMEGA328P_TQFP, U2 USD-SOCKETSMD, U3 3.3V/150mA, U4 9DoF IMU, Y1 16MHz

Commit message: Added pressure sensor for gits and giggles.
Parts:
- added U5: BME280, femtosat:LGA-8-2.5X2.5
- moved D1 5.68 mm to (40.6, 20.3), turned to 270 degrees
- moved R1 4.02 mm to (39.4, 20.3), turned to 270 degrees
Connections:
- net 3.3V: now also U5.2, U5.6, U5.8
- net GND: now also U5.1, U5.5, U5.7
- net SCL: now also U5.4
- net SDA: now also U5.3
Routing:
- net SDA: track 25.2 -> 40.4 mm, vias 2 -> 3
- net SCL: track 29.9 -> 45.0 mm, vias 2 -> 3
- net 3.3V: track 138.1 -> 149.3 mm
Changed lines of the file:
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@@
 <attribute name="DIGIKEY" value="311-1343-1-ND " x="2.54" y="11.43" size="1.778" layer="27" rot="R90" display="off"/>
 </element>
-<element name="D1" library="femtosat" package="LED-0603" value="RED" x="35.56" y="22.86">
-<attribute name="DIGIKEY" value="160-1181-1-ND" x="35.56" y="22.86" size="1.778" layer="27" display="off"/>
+<element name="D1" library="femtosat" package="LED-0603" value="RED" x="40.64" y="20.32" rot="R270">
+<attribute name="DIGIKEY" value="160-1181-1-ND" x="40.64" y="20.32" size="1.778" layer="27" rot="R270" display="off"/>
 </element>
 <element name="J1" library="SparkFun-Connectors" package="1X02" value="" x="8.255" y="8.3058"/>
@@
 <element name="J5" library="SparkFun-Connectors" package="1X02" value="" x="16.51" y="21.59" rot="R270"/>
 <element name="J6" library="SparkFun-Connectors" package="1X02" value="" x="8.89" y="21.59" rot="R270"/>
-<element name="R1" library="femtosat" package="0603" value="330" x="35.56" y="21.59">
-<attribute name="DIGIKEY" value="311-330GRCT-ND " x="35.56" y="21.59" size="1.778" layer="27" display="off"/>
+<element name="R1" library="femtosat" package="0603" value="330" x="39.37" y="20.32" rot="R270">
+<attribute name="DIGIKEY" value="311-330GRCT-ND " x="39.37" y="20.32" size="1.778" layer="27" rot="R270" display="off"/>
 </element>
 <element name="R2" library="femtosat" package="0603-RES" value="10K" x="2.54" y="15.24" rot="R90">
@@
 <element name="J7" library="SparkFun-Connectors" package="1X02" value="" x="8.2296" y="14.9098" rot="R270"/>
 <element name="J8" library="SparkFun-Connectors" package="1X02" value="" x="8.3312" y="3.7084"/>
+<element name="U5" library="femtosat" package="LGA-8-2.5X2.5" value="BME280" x="34.29" y="22.86" rot="R270">
+<attribute name="DIGIKEY" value="828-1063-1-ND " x="34.29" y="22.86" size="1.016" layer="27" rot="R270" display="off"/>
+</element>
 </elements>
 <signals>
@@
 <via x="21.59" y="8.89" extent="1-16" drill="0.508"/>
 <wire x1="15.24" y1="8.89" x2="21.59" y2="8.89" width="0.635" layer="16"/>
+<contactref element="U5" pad="1"/>
+<contactref element="U5" pad="7"/>
+<contactref element="U5" pad="5"/>
 </signal>
 <signal name="3.3V">
@@
 <wire x1="28.01094375" y1="19.134125" x2="28.01094375" y2="11.43" width="0.381" layer="1"/>
 <wire x1="28.01094375" y1="11.43" x2="28.01094375" y2="11.239703125" width="0.381" layer="1"/>
-<wire x1="25.08110625" y1="26.5223" x2="27.0157" y2="24.30830625" width="0.381" layer="1"/>
+<wire x1="27.0157" y1="24.30830625" x2="25.08110625" y2="26.5223" width="0.381" layer="1"/>
 <wire x1="27.0157" y1="24.30830625" x2="27.0157" y2="20.12936875" width="0.381" layer="1"/>
 <wire x1="27.0157" y1="20.12936875" x2="28.01094375" y2="19.134125" width="0.381" layer="1"/>
@@
 <wire x1="23.9522" y1="21.6662" x2="24.0002" y2="21.7142" width="0.254" layer="1"/>
 <wire x1="24.0002" y1="21.7142" x2="24.0002" y2="22.5044" width="0.254" layer="1"/>
+<contactref element="U5" pad="8"/>
+<contactref element="U5" pad="6"/>
+<contactref element="U5" pad="2"/>
+<wire x1="33.56" y1="24.13" x2="33.265" y2="23.835" width="0.254" layer="1"/>
+<wire x1="33.56" y1="24.13" x2="34.29" y2="24.13" width="0.254" layer="1"/>
+<wire x1="34.29" y1="23.185" x2="34.29" y2="24.13" width="0.254" layer="1"/>
+<wire x1="34.29" y1="23.185" x2="35.315" y2="23.185" width="0.254" layer="1"/>
+<wire x1="34.29" y1="22.535" x2="33.265" y2="22.535" width="0.254" layer="1"/>
+<wire x1="34.29" y1="22.535" x2="34.29" y2="23.185" width="0.254" layer="1"/>
+<wire x1="33.265" y1="23.835" x2="32.79169375" y2="24.30830625" width="0.254" layer="1"/>
+<wire x1="32.79169375" y1="24.30830625" x2="27.0157" y2="24.30830625" width="0.254" layer="1"/>
 </signal>
 <signal name="MISO">
@@
 <wire x1="19.9" y1="24.13" x2="25.4" y2="24.13" width="0.254" layer="1"/>
 <wire x1="25.4" y1="24.13" x2="25.4" y2="17.78" width="0.254" layer="1"/>
-<wire x1="25.4" y1="17.78" x2="22.479" y2="14.859" width="0.254" layer="16"/>
+<wire x1="22.479" y1="14.859" x2="25.4" y2="17.78" width="0.254" layer="16"/>
 <wire x1="19.177" y1="14.859" x2="22.479" y2="14.859" width="0.254" layer="16"/>
 <via x="19.177" y="14.859" extent="1-16" drill="0.35"/>
@@
 <wire x1="20.6732" y1="12.773853125" x2="19.91359375" y2="13.533459375" width="0.254" layer="1"/>
 <wire x1="19.91359375" y1="13.533459375" x2="19.91359375" y2="14.12240625" width="0.254" layer="1"/>
+<contactref element="U5" pad="3"/>
+<wire x1="25.4" y1="17.78" x2="31.75" y2="17.78" width="0.254" layer="16"/>
+<wire x1="31.75" y1="17.78" x2="36.83" y2="22.86" width="0.254" layer="16"/>
+<via x="36.83" y="22.86" extent="1-16" drill="0.35"/>
+<wire x1="36.83" y1="22.86" x2="36.505" y2="22.535" width="0.254" layer="1"/>
+<wire x1="36.505" y1="22.535" x2="35.315" y2="22.535" width="0.254" layer="1"/>
 </signal>
 <signal name="SCL">
@@
 <wire x1="26.0576" y1="17.5076125" x2="25.4" y2="16.8500125" width="0.254" layer="1"/>
 <wire x1="26.0576" y1="24.0471375" x2="26.0576" y2="17.5076125" width="0.254" layer="1"/>
-<wire x1="25.4" y1="16.51" x2="22.987" y2="14.097" width="0.254" layer="16"/>
+<wire x1="22.987" y1="14.097" x2="25.4" y2="16.51" width="0.254" layer="16"/>
 <wire x1="22.987" y1="14.097" x2="18.288" y2="14.097" width="0.254" layer="16"/>
 <via x="18.288" y="14.097" extent="1-16" drill="0.35"/>
@@
 <wire x1="19.9" y1="25.654" x2="21.7424" y2="25.654" width="0.254" layer="1"/>
 <wire x1="21.7424" y1="25.654" x2="22.86" y2="24.5364" width="0.254" layer="1"/>
+<contactref element="U5" pad="4"/>
+<wire x1="25.4" y1="16.51" x2="26.2636" y2="17.3736" width="0.254" layer="16"/>
+<wire x1="36.1347375" y1="21.59" x2="36.83" y2="21.59" width="0.254" layer="16"/>
+<wire x1="31.9183375" y1="17.3736" x2="36.1347375" y2="21.59" width="0.254" layer="16"/>
+<via x="36.83" y="21.59" extent="1-16" drill="0.35"/>
+<wire x1="36.83" y1="21.59" x2="36.535" y2="21.885" width="0.254" layer="1"/>
+<wire x1="36.535" y1="21.885" x2="35.315" y2="21.885" width="0.254" layer="1"/>
+<wire x1="26.2636" y1="17.3736" x2="31.9183375" y2="17.3736" width="0.254" layer="16"/>
 </signal>
 <signal name="N$4">
@@
 <contactref element="D1" pad="A"/>
 <contactref element="R1" pad="1"/>
-<wire x1="34.71" y1="21.59" x2="34.683" y2="21.617" width="0.254" layer="1"/>
-<wire x1="34.683" y1="21.617" x2="34.683" y2="22.86" width="0.254" layer="1"/>
+<wire x1="39.37" y1="21.17" x2="40.613" y2="21.17" width="0.254" layer="1"/>
+<wire x1="40.613" y1="21.17" x2="40.64" y2="21.197" width="0.254" layer="1"/>
 </signal>
 <signal name="IO5">
@@
 <wire x1="36.83" y1="12.8877" x2="36.83" y2="19.05" width="0.254" layer="16"/>
 <via x="36.83" y="19.05" extent="1-16" drill="0.35"/>
-<wire x1="36.83" y1="19.05" x2="36.41" y2="19.47" width="0.254" layer="1"/>
-<wire x1="36.41" y1="19.47" x2="36.41" y2="21.59" width="0.254" layer="1"/>
 <wire x1="23.915425" y1="3.874771875" x2="25.062496875" y2="2.7277" width="0.254" layer="1"/>
 <wire x1="25.062496875" y1="2.7277" x2="26.67" y2="2.7277" width="0.254" layer="1"/>
+<wire x1="36.83" y1="19.05" x2="38.95" y2="19.05" width="0.254" layer="1"/>
+<wire x1="38.95" y1="19.05" x2="39.37" y2="19.47" width="0.254" layer="1"/>
 </signal>
 <signal name="RXD">
